File: MonitorWizard-Logger.sch (EAGLE design)
At the start: 59 parts, among them SW1 ACTION, T1 FDN340P, U1 NCP1117ST50T3G, U2 LP2985-33DBVR, U4-NRF24L01 NRF24L01+-PCB-AERIAL, U5 LMV358IDGKR, U6 ATMEGA328P-PU, U7 RFM69CW, X3 POWERSUPPLY_DC21MMX, Y2 CSTCE16M0V53-R0 16MHZ, Y3 32.768kHz

Commit message: Switch to PNP transistors, connect data lines to chip.
Parts:
- removed T2, T3: (no value), transistor:BC337-NPN-TO92-CBE
- added Q1, Q2: 2N3906, transistor-pnp:2N3906
- added R4, R5, R6, R7, R8, R9: (no value), rcl:R-EU_0207/10
Connections:
- removed net BTN0: U6.(INT0)PD2
- removed net PROC_GND: C12.1, C13.1, ICSP2.6, JP1.CTS, JP1.GND, PROC_CURRENT.P$1, U6.AGND, U6.GND
- removed net RFMODULE_GND: T2.C, U4-NRF24L01.GND, U7.GND@1, U7.GND@2
- removed net SENSOR_GND: T3.C
- new net CHIP_SS: R7.1, U6.(SS)PB2
- new net INT0: R9.1, U6.(INT0)PD2
- new net N$8: Q2.E, SENSOR_CURRENT.P$2
- net GND: now also C12.1, C13.1, ICSP2.6, JP1.CTS, JP1.GND, PROC_CURRENT.P$1, U4-NRF24L01.GND, U6.AGND, U6.GND, U7.GND@1, U7.GND@2; no longer RF_CURRENT.P$2, SENSOR_CURRENT.P$2
- net MISO1: now also R5.1
- net MOSI1: now also R6.1
- net N$2: now also Q1.B, R1.2; no longer RF_CURRENT.P$1, T2.E
- net N$4: now also Q2.B, R3.2; no longer R1.2, T2.B
- net N$5: now also Q1.E, RF_CURRENT.P$2; no longer SENSOR_CURRENT.P$1, T3.E
- net N$6: now also R8.1, U6.(AIN0)PD6; no longer R3.2, T3.B
- net RFMODULE_CS: now also R7.2
- net RFMODULE_MISC1: now also R8.2
- net RFMODULE_MISC2: now also R9.2
- net RFMODULE_MISO: now also R5.2
- net RFMODULE_MOSI: now also R6.2
- net RFMODULE_POWER_ON: now also U6.(ICP)PB0
- net RFMODULE_SCK: now also R4.2
- net SCK1: now also R4.1
- net SENSOR_POWER_ON: now also U6.(OC1)PB1
- net VBAT: now also RF_CURRENT.P$1, SENSOR_CURRENT.P$1
Other:
- moved on the sheet: GND, R1, R3, VBAT

Commit message: Remove redundant components, play with board layout.
Parts:
- removed AD: 6x1F-H8.5, SmartPrj:PINHD-1X6
- removed C1, C2, C4, C5, C6: 100n, SmartPrj:C-EU0603-RND
- removed C3: 1u, SmartPrj:C-EU0603-RND
- removed D1: M7, diode:DIODE-SMB
- removed D2: CD1206-S01575, diode:DIODE-MINIMELF
- removed ICSP: 3x2 M, SmartPrj:PINHD-2X3
- removed IOH1: 10x1F-H8.5, SmartPrj:PINHD-1X10_ARD
- removed IOL, POWER: 8x1F-H8.5, SmartPrj:PINHD-1X8
- removed JP2: 2x2 M - NM, SmartPrj:PINHD-2X2
- removed L, RX, TX: YELLOW, led:LEDCHIP-LED0805
- removed ON: GREEN, led:LEDCHIP-LED0805
- removed PC1, PC2: 47u, rcl:CPOL-EUD
- removed PROC_CURRENT: CURRENT_MEASURE_0.4A, Probes:CURRENT_MEASURE_0.4A
- removed R2: 1M, SmartPrj:R-EU_R0603
- removed RESET: TS42031-160R-TR-7260, SmartPrj:TS42
- removed RESET-EN: (no value), jumper:SJ
- removed RN1: 10K, resistor-dil:4R-NCAY16
- removed RN2, RN4: 1K, resistor-dil:4R-NCAY16
- removed RN3: 22R, resistor-dil:4R-NCAY16
- removed T1: FDN340P, zetex:PMOSSOT23
- removed U1: NCP1117ST50T3G, linear:MC33269ST-3.3T3
- removed U2: LP2985-33DBVR, SmartPrj:LP2985-XXDBVR33
- removed U5: LMV358IDGKR, linear:LMV358MMX
- removed Y2: CSTCE16M0V53-R0 16MHZ, SmartPrj:RESONATORMU
- removed ZU4: ATMEGA328P-PU, SmartPrj:ATMEGA328P-PU
Connections:
- removed net +3V3: C3.2, POWER.4, U2.OUT, U5A.-IN
- removed net AD0: AD.1, ZU4.(ADC0)PC0)
- removed net AD1: AD.2, ZU4.(ADC1)PC1
- removed net AD2: AD.3, ZU4.(ADC2)PC2
- removed net AD3: AD.4, ZU4.(ADC3)PC3
- removed net AD4/SDA: AD.5, IOH1.9, ZU4.(ADC4)PC4
- removed net AD5/SCL: AD.6, IOH1.10, ZU4.(ADC5)PC5
- removed net CMP: RN1A.1, RN1B.1, U5A.+IN
- removed net DTR: C5.1, RN2D.1
- removed net GATE_CMD: T1.G, U5A.OUT
- removed net IO0: IOL.1, RN4B.1, ZU4.(RXD)PD0
- removed net IO1: IOL.2, RN4A.1, ZU4.(TXD)PD1
- removed net IO2: IOL.3, ZU4.(INT0)PD2
- removed net IO3: IOL.4, ZU4.(INT1)PD3
- removed net IO4: IOL.5, ZU4.(T0)PD4
- removed net IO5: IOL.6, ZU4.(T1)PD5
- removed net IO6: IOL.7, ZU4.(AIN0)PD6
- removed net IO7: IOL.8, ZU4.(AIN1)PD7
- removed net IO8: IOH1.1, ZU4.(ICP)PB0
- removed net IO9: IOH1.2, ZU4.(OC1)PB1
- removed net L13: RN2A.2, U5B.-IN, U5B.OUT
- removed net M8RXD: RN4B.2
- removed net M8TXD: RN4A.2
- removed net MISO: ICSP.1, IOH1.5, ZU4.(MISO)PB4
- removed net MOSI: ICSP.4, IOH1.4, ZU4.(MOSI)PB3
- removed net N$1: L.A, RN2A.1
- removed net N$3: ON.A, RN4C.2, RN4D.2
- removed net N$35: RN2B.2, RX.A
- removed net N$36: RN2C.2, TX.A
- removed net PB4: JP2.1
- removed net PB5: JP2.3
- removed net PB6: JP2.2
- removed net PB7: JP2.4
- removed net PWRIN: D1.A
- removed net RESET: C5.2, D2.A, ICSP.5, POWER.3, RESET-EN.1, RESET-EN.2, RESET.3, RESET.4, RN1D.1, ZU4.RESET
- removed net RXLED: RX.C
- removed net SCK: ICSP.3, IOH1.6, U5B.+IN, ZU4.(SCK)PB5
- removed net SS: IOH1.3, ZU4.(SS)PB2
- removed net TXLED: TX.C
- removed net USBVCC: T1.D
- removed net VIN: D1.C, PC1.+, POWER.8, RN1A.2, U1.IN
- removed net XTAL1: R2.1, Y2.3, ZU4.XTAL1
- removed net XTAL2: R2.2, Y2.1, ZU4.XTAL2
- net +5V: no longer C1.2, C2.2, C6.2, D2.C, ICSP.2, PC2.+, POWER.2, POWER.5, RN1D.2, RN2B.1, RN2C.1, RN4C.1, RN4D.1, T1.S, U1.OUT, U1.OUT@1, U2.IN, U2.ON/!OFF, U5P.V+, ZU4.AVCC, ZU4.VCC
- net AREF: no longer C4.2, IOH1.8, ZU4.AREF
- net GND: no longer C1.1, C2.1, C3.1, C4.1, C6.1, ICSP.6, IOH1.7, L.C, ON.C, PC1.-, PC2.-, POWER.6, POWER.7, PROC_CURRENT.P$1, PROC_CURRENT.P$2, RESET.1, RESET.2, RN1B.2, RN2D.2, U1.GND/ADJ, U2.GND, U5P.V-, Y2.2, ZU4.AGND, ZU4.GND
Other:
- note added: "Fiducials"
- note removed: "0"
- note removed: "1"
- note removed: "10"
- note removed: "11"
- note removed: "12"
- note removed: "13"
- note removed: "2"
- note removed: "3"
- note removed: "4"
- note removed: "5"
- note removed: "6"
- note removed: "7"
- note removed: "8"
- note removed: "9"
- note removed: "Arduino(TM) UNO Rev3"
- note removed: "ONLY IF CC!!!!!!! 2N5551 or equivalent: http://uk.farnell.com/fairchild-semiconductor/2n5551/transistor-npn-160v-to-92/dp/9846751 or cheaper http://uk.farnell.com/multicomp/2n4401/transistor-npn-to-92/dp/1574373 ONLY when using CC 7segs. When using CA, use a NPN transistor instead!"
- note removed: "SCL"
- note removed: "SDA"
- note removed: "USB boot En"
- note removed: "Use of the ARDUINO name must be compliant with http://www.arduino.cc/en/Main/Policy"

Commit message: Add DHT22 library, tweak board layout. Still unfinished.
Parts:
- added D1: 1N4148DO35-10, diode:1N4148DO35-10
- added R2: 10K, resistor:R-EU_0207/10
- added U1: DHT22, RHT03_DHT-22_AM2302:RHT03_DHT-22_AM2302
- U3: value (none) -> 7805-TO220
Connections:
- removed net N$7: U3.OUT
- new net 5V_REG: D1.A, U3.OUT
- new net DHT22_DATA: R2.1, U1.DATA, U6.(ADC0)PC0)
- new net SENSOR_3V3: R2.2, U1.VDD
- net GND: now also U1.GND
- net VBAT: now also D1.C
Other:
- note added: "Are NPNs on the ground side, or PNPs on the positive side better? NPNs are more efficient, but the voltage across the transistor or shunt may lead to issues with signals or regulators. Hence PNPs are used"
- note added: "Note: Arduino power might be higher voltage than 3V3 - should signal 1 to the device by just not driving it low (pullup resistor does the work)."
- note added: "TODO: Something clever here that causes the transistor to additionally work as a controllable 3.3V regulator, whilst not adding any leakage current when off?"
- note added: "takes 3-5v, no need for regulator?"
- note removed: "Are NPNs on the ground side, or PNPs on the positive side better? NPNs are more efficient, but the voltage across the transistor or shunt may lead to issues with signals or regulators."
Changed lines of the file:
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@@
 <part name="R1" library="resistor" deviceset="R-EU_" device="0207/10"/>
 <part name="R3" library="resistor" deviceset="R-EU_" device="0207/10"/>
-<part name="U3" library="SparkFun-PowerIC" deviceset="V_REG_78XX" device="-TO-220"/>
+<part name="U3" library="SparkFun-PowerIC" deviceset="V_REG_78XX" device="-TO-220" value="7805-TO220"/>
 <part name="Q1" library="transistor-pnp" deviceset="2N3906" device=""/>
 <part name="Q2" library="transistor-pnp" deviceset="2N3906" device=""/>
@@
 <part name="R8" library="rcl" deviceset="R-EU_" device="0207/10"/>
 <part name="R9" library="rcl" deviceset="R-EU_" device="0207/10"/>
+<part name="U1" library="RHT03_DHT-22_AM2302" deviceset="RHT03_DHT-22_AM2302" device="" value="DHT22"/>
+<part name="R2" library="resistor" deviceset="R-EU_" device="0207/10" value="10K"/>
+<part name="D1" library="diode" deviceset="1N4148" device="DO35-10"/>
 </parts>
 <sheets>
@@
 <text x="421.64" y="-378.46" size="1.778" layer="94">(RF Module)</text>
 <text x="482.6" y="-378.46" size="1.778" layer="94">(Sensor Modules)</text>
-<wire x1="464.82" y1="-386.08" x2="464.82" y2="-368.3" width="0.1524" layer="94"/>
-<wire x1="464.82" y1="-368.3" x2="510.54" y2="-368.3" width="0.1524" layer="94"/>
+<wire x1="477.52" y1="-386.08" x2="477.52" y2="-368.3" width="0.1524" layer="94"/>
+<wire x1="477.52" y1="-368.3" x2="510.54" y2="-368.3" width="0.1524" layer="94"/>
 <wire x1="510.54" y1="-368.3" x2="510.54" y2="-386.08" width="0.1524" layer="94"/>
-<wire x1="510.54" y1="-386.08" x2="464.82" y2="-386.08" width="0.1524" layer="94"/>
+<wire x1="510.54" y1="-386.08" x2="477.52" y2="-386.08" width="0.1524" layer="94"/>
 <wire x1="414.02" y1="-368.3" x2="414.02" y2="-386.08" width="0.1524" layer="94"/>
 <wire x1="414.02" y1="-386.08" x2="444.5" y2="-386.08" width="0.1524" layer="94"/>
@@
 <wire x1="444.5" y1="-368.3" x2="414.02" y2="-368.3" width="0.1524" layer="94"/>
 <text x="543.56" y="-330.2" size="1.778" layer="97">Are NPNs on the ground side, or PNPs on the positive side better?
-NPNs are more efficient, but the voltage across the transistor or shunt may lead to issues with signals or regulators.</text>
+NPNs are more efficient, but the voltage across the transistor or shunt may lead to issues with signals or regulators.
+Hence PNPs are used</text>
 <text x="533.4" y="-299.72" size="1.778" layer="97">Battery Contact(s)</text>
 <text x="581.66" y="-76.2" size="1.778" layer="94">Fiducials</text>
+<text x="165.1" y="-368.3" size="1.778" layer="97">takes 3-5v, no need for regulator?</text>
+<text x="383.54" y="-353.06" size="1.778" layer="94">TODO: Something clever here that causes the transistor to additionally work as a controllable 3.3V
+ regulator, whilst not adding any leakage current when off?</text>
+<text x="203.2" y="-162.56" size="1.778" layer="94">Note: Arduino power might be higher voltage than 3V3 - should signal 1 to the device by just not driving it low (pullup resistor does the work).</text>
 </plain>
 <instances>
@@
 <instance part="R8" gate="G$1" x="236.22" y="-170.18"/>
 <instance part="R9" gate="G$1" x="236.22" y="-172.72"/>
+<instance part="U1" gate="G$1" x="154.94" y="-365.76"/>
+<instance part="R2" gate="G$1" x="119.38" y="-355.6" rot="R90"/>
+<instance part="D1" gate="G$1" x="388.62" y="-302.26"/>
 </instances>
 <busses>
@@
 </segment>
 <segment>
-<wire x1="193.04" y1="-398.78" x2="81.28" y2="-398.78" width="0.1524" layer="91"/>
+<wire x1="193.04" y1="-398.78" x2="124.46" y2="-398.78" width="0.1524" layer="91"/>
 <label x="109.22" y="-398.78" size="1.778" layer="95"/>
+<pinref part="U1" gate="G$1" pin="GND"/>
+<wire x1="124.46" y1="-398.78" x2="81.28" y2="-398.78" width="0.1524" layer="91"/>
+<wire x1="144.78" y1="-373.38" x2="124.46" y2="-373.38" width="0.1524" layer="91"/>
+<wire x1="124.46" y1="-373.38" x2="124.46" y2="-398.78" width="0.1524" layer="91"/>
+<junction x="124.46" y="-398.78"/>
 </segment>
 </net>
@@
 <segment>
 <label x="416.56" y="-302.26" size="1.778" layer="95"/>
-<wire x1="416.56" y1="-302.26" x2="439.42" y2="-302.26" width="0.1524" layer="91"/>
+<wire x1="391.16" y1="-302.26" x2="439.42" y2="-302.26" width="0.1524" layer="91"/>
 <pinref part="RF_CURRENT" gate="G$1" pin="P$1"/>
 <pinref part="SENSOR_CURRENT" gate="G$1" pin="P$1"/>
@@
 <junction x="528.32" y="-302.26"/>
 <junction x="523.24" y="-302.26"/>
+<pinref part="D1" gate="G$1" pin="C"/>
 </segment>
 </net>
@@
 </segment>
 </net>
-<net name="N$7" class="0">
+<net name="5V_REG" class="0">
 <segment>
 <pinref part="U3" gate="G$1" pin="OUT"/>
-<wire x1="363.22" y1="-302.26" x2="373.38" y2="-302.26" width="0.1524" layer="91"/>
+<wire x1="363.22" y1="-302.26" x2="386.08" y2="-302.26" width="0.1524" layer="91"/>
 <label x="368.3" y="-302.26" size="1.778" layer="95"/>
+<pinref part="D1" gate="G$1" pin="A"/>
 </segment>
 </net>
@@
 </segment>
 <segment>
-<wire x1="88.9" y1="-332.74" x2="129.54" y2="-332.74" width="0.1524" layer="91"/>
+<wire x1="88.9" y1="-332.74" x2="119.38" y2="-332.74" width="0.1524" layer="91"/>
 <label x="101.6" y="-330.2" size="1.778" layer="95"/>
+<pinref part="U1" gate="G$1" pin="VDD"/>
+<wire x1="119.38" y1="-332.74" x2="124.46" y2="-332.74" width="0.1524" layer="91"/>
+<wire x1="124.46" y1="-332.74" x2="129.54" y2="-332.74" width="0.1524" layer="91"/>
+<wire x1="144.78" y1="-358.14" x2="124.46" y2="-358.14" width="0.1524" layer="91"/>
+<wire x1="124.46" y1="-358.14" x2="124.46" y2="-332.74" width="0.1524" layer="91"/>
+<junction x="124.46" y="-332.74"/>
+<pinref part="R2" gate="G$1" pin="2"/>
+<wire x1="119.38" y1="-350.52" x2="119.38" y2="-332.74" width="0.1524" layer="91"/>
+<junction x="119.38" y="-332.74"/>
 </segment>
 </net>
@@
 </segment>
 </net>
+<net name="DHT22_DATA" class="0">
+<segment>
+<pinref part="U1" gate="G$1" pin="DATA"/>
+<pinref part="R2" gate="G$1" pin="1"/>
+<wire x1="144.78" y1="-363.22" x2="119.38" y2="-363.22" width="0.1524" layer="91"/>
+<wire x1="119.38" y1="-363.22" x2="119.38" y2="-360.68" width="0.1524" layer="91"/>
+<wire x1="119.38" y1="-363.22" x2="83.82" y2="-363.22" width="0.1524" layer="91"/>
+<junction x="119.38" y="-363.22"/>
+<label x="91.44" y="-363.22" size="1.778" layer="95"/>
+</segment>
+<segment>
+<pinref part="U6" gate="G$1" pin="(ADC0)PC0)"/>
+<wire x1="167.64" y1="-162.56" x2="200.66" y2="-162.56" width="0.1524" layer="91"/>
+<label x="185.42" y="-162.56" size="1.778" layer="95"/>
+</segment>
+</net>

Commit message: Replace power supply with low power switching setup. Remove resistors for level shifting, since everything will now be running at 3.3v.
Parts:
- removed D1: 1N4148DO35-10, diode:1N4148DO35-10
- removed Q1, Q2: 2N3906, transistor-pnp:2N3906
- removed R4, R5, R6, R7, R8, R9: (no value), rcl:R-EU_0207/10
- removed U7: RFM69CW, SparkFun-RF:RFM69CW
- added C1: 10uH, rcl:C-EU025-024X044
- added C2: 2.2uH, rcl:C-EU025-024X044
- added L1: 10uH, InductorsThru:MURATA-1100R
- added U2: RFM69HW, SparkFun-RF:RFM69HW
- R2: value 10K -> (none)
- R3: value (none) -> 10K
- U3: value 7805-TO220 -> LTC3531; device SparkFun-PowerIC:V_REG_78XX-TO-220 -> linear-sen:LTC3531
Connections:
- removed net 5V_REG: D1.A, U3.OUT
- removed net CHIP_SS: R7.1, U6.(SS)PB2
- removed net INT0: R9.1, U6.(INT0)PD2
- removed net N$4: Q2.B, R3.2
- removed net N$5: Q1.E, RF_CURRENT.P$2
- removed net N$6: R8.1, U6.(AIN0)PD6
- removed net N$8: Q2.E, SENSOR_CURRENT.P$2
- removed net RFMODULE_POWER_ON: R1.1, U6.(ICP)PB0
- removed net SENSOR_POWER_ON: R3.1, U6.(OC1)PB1
- new net 3V3: C1.1, R2.2, RF_CURRENT.P$1, U3.VOUT
- new net N$1: L1.2, U3.SW2
- new net N$3: R1.2, R2.1, U3.FB
- new net RF_SS: U6.(SS)PB2
- new net SENSOR_POWER: SENSOR_CURRENT.P$1, U6.(OC1)PB1
- net DHT22_DATA: now also R3.1; no longer R2.1
- net GND: now also C1.2, C2.2, R1.1, U2.GND@1, U2.GND@2; no longer U7.GND@1, U7.GND@2
- net MISO1: no longer R5.1
- net MOSI1: no longer R6.1
- net N$2: now also L1.1, U3.SW1; no longer Q1.B, R1.2
- net N$9: now also U2.ANT; no longer U7.ANT
- net RFMODULE_3V3: now also RF_CURRENT.P$2, U2.3.3V; no longer U7.3.3V
- net RFMODULE_CS: now also U2.NSS; no longer R7.2, U7.NSS
- net RFMODULE_MISC1: now also U2.RESET, U6.(AIN0)PD6; no longer R8.2, U7.RESET
- net RFMODULE_MISC2: now also U2.DIO0, U6.(INT0)PD2; no longer R9.2, U7.DIO0
- net RFMODULE_MISO: now also U2.MISO; no longer R5.2, U7.MISO
- net RFMODULE_MOSI: now also U2.MOSI; no longer R6.2, U7.MOSI
- net RFMODULE_SCK: now also U2.SCK; no longer R4.2, U7.SCK
- net SCK1: no longer R4.1
- net SENSOR_3V3: now also R3.2, SENSOR_CURRENT.P$2; no longer R2.2
- net VBAT: now also C2.1, U3.!SHDN, U3.VIN; no longer D1.C, RF_CURRENT.P$1, SENSOR_CURRENT.P$1
- net VBJ: no longer U3.IN
Other:
- note added: "Barrel jack voltage dropped to 3V3 through a 3V3 linear regulator. When powered from a barrel jack, wasted current isn't a huge deal - linear regulator OK. Diode to prevent leakage?"
- note added: "LTC3531EDD#PBF is leadfree adjustible version in 8-pin package (Farnell OC 1663711) Better to neglect the feedback, use the fixed 3.3v, and buy from Rapid: 59-4951 http://www.rapidonline.com/electronic-components/linear-tech-ltc3531edd-3-3-pbf-dc-dc-converter-ic-dfn-8-pin-59-4951"
- note added: "TODO decouple 2.2u on in 10u on out"
- note added: "With fixed output, this is not connected and should not be populated. With adjustible versions, the output voltage can be adjusted from 2V to 5V. Vout = 1.225 ( 1 + r2/r1) where r2 is between vout and fb, and r1 is from fb to gnd"
- note removed: "Are NPNs on the ground side, or PNPs on the positive side better? NPNs are more efficient, but the voltage across the transistor or shunt may lead to issues with signals or regulators. Hence PNPs are used"
- note removed: "Barrel jack voltage dropped to 3V3 or 4V? When powered from a barrel jack, wasted current isn't a huge deal - linear regulator OK. Diode to prevent leakage."
- moved on the sheet: R1, R2, R3

Commit message: Add SD card, battery box. Nearly finished - just have to connect SD and lay out.
Parts:
- added CON1: MICROSD, adafruit:MICROSD
- added IC1: LD117AV33, v-reg:LD117AV33
- added U$1: SDMMC06132, adafruit:SDMMC06132
- added U$2: 2464, keystone:2464
Connections:
- removed net VCC: C13.2, U6.AVCC, U6.VCC
- new net SD_CS: CON1.CS, U$1.CS
- new net SD_DAT1: CON1.DAT1, U$1.DAT1
- new net SD_DAT2: CON1.DAT2, U$1.DAT2
- new net SD_DIN: CON1.DATA_IN, U$1.DATA_IN
- new net SD_DO: CON1.DATA_OUT, U$1.DATA_OUT
- new net SD_SCLK: CON1.SCLK, U$1.SCLK
- net 3V3: now also C13.2, CON1.VDD, IC1.OUT, U$1.VDD, U6.AVCC, U6.VCC
- net GND: now also CON1.GND, CON1.GND1, CON1.VSS, IC1.ADJ, U$1.GND, U$1.VSS1, U$1.VSS2, U$2.-
- net VBAT: now also U$2.+
- net VBJ: now also IC1.IN
Other:
- note added: "Farnell 1654360"
- note added: "Farnell 9755837"
- note added: "Keystone 2464 Farnell 1704231"
- note added: "OC Farnell 2062671"
- note added: "SD Card - Micro and Regular footprints in parallel"
- note added: "Storage"
- note added: "electrolytic?"
- note removed: "TODO decouple 2.2u on in 10u on out"
- note removed: "TODO: Something clever here that causes the transistor to additionally work as a controllable 3.3V regulator, whilst not adding any leakage current when off?"

Commit message: Hopefully completed the schematic.
Parts:
- removed SW1: ACTION, switch-omron:10-XX
- added J1, J2, J3: 22-27-2041-04, con-molex:22-27-2041-04
- added R4: TBD, resistor:R-EU_0207/10
Connections:
- net SENSOR_POWER renamed EXT_SENSOR_POWER
- removed net RFMODULE_MISO: U2.MISO, U4-NRF24L01.MISO
- removed net RFMODULE_MOSI: U2.MOSI, U4-NRF24L01.MOSI
- removed net RFMODULE_SCK: U2.SCK, U4-NRF24L01.SCK
- removed net RF_SS: U6.(SS)PB2
- removed net SD_DIN: CON1.DATA_IN, U$1.DATA_IN
- removed net SD_DO: CON1.DATA_OUT, U$1.DATA_OUT
- removed net SD_SCLK: CON1.SCLK, U$1.SCLK
- removed net SENSOR_3V3: R3.2, SENSOR_CURRENT.P$2, U1.VDD
- new net DHT22_3V3: R3.2, U1.VDD, U6.(AIN1)PD7
- new net EXT_ANALOG_0_TIM: J1-2.S, U6.(ADC0)PC0), U6.(T1)PD5
- new net EXT_ANALOG_1: J1-3.S, U6.(ADC1)PC1
- new net EXT_ANALOG_2: J2-2.S, U6.(ADC2)PC2
- new net EXT_ANALOG_3: J2-3.S, U6.(ADC3)PC3
- new net EXT_ANALOG_4: J3-2.S, U6.(ADC4)PC4
- new net EXT_ANALOG_5: J3-3.S, U6.(ADC5)PC5
- new net EXT_SENSOR_3V3: J1-1.S, J2-1.S, J3-1.S, R4.1, SENSOR_CURRENT.P$2
- new net RFMODULE_MISC2_INT: U2.DIO0, U4-NRF24L01.IRQ
- new net SD_DETECT: CON1.CARD_DETECT, U$1.CARD_DETECT, U6.(INT1)PD3
- net AREF: now also R4.2
- net DHT22_DATA: now also U6.(T0)PD4; no longer U6.(ADC0)PC0)
- net GND: now also CON1.CARD_DETECT1, J1-4.S, J2-4.S, J3-4.S, U$1.COMMON_SW; no longer SW1.S, SW1.S1
- net MISO1: now also CON1.DATA_OUT, U$1.DATA_OUT, U2.MISO, U4-NRF24L01.MISO
- net MOSI1: now also CON1.DATA_IN, U$1.DATA_IN, U2.MOSI, U4-NRF24L01.MOSI
- net RFMODULE_CS: now also U6.(SS)PB2
- net RFMODULE_MISC2: no longer U2.DIO0, U4-NRF24L01.IRQ
- net SCK1: now also CON1.SCLK, U$1.SCLK, U2.SCK, U4-NRF24L01.SCK
- net SD_CS: now also U6.(ICP)PB0
Other:
- note added: "DAT1/DAT2 used for high speed comms only"
- note added: "Farnell 1654360 NO LONGER STOCKED CHECK COMPATIBILITY: 2424133"
- note added: "RF module uses little current in low power mode - no need to disconnect"
- note removed: "Farnell 1654360"

Commit message: Add decoupling capacitors, begin to route board.
Parts:
- added C3, C4, C5, C6, C7: 0.1u, rcl:C-EU025-024X044
Connections:
- net EXT_SENSOR_POWER renamed SENSOR_POWER
- removed net +5V: ICSP2.2
- removed net DHT22_3V3: R3.2, U1.VDD, U6.(AIN1)PD7
- removed net EXT_SENSOR_3V3: J1-1.S, J2-1.S, J3-1.S, R4.1, SENSOR_CURRENT.P$2
- removed net RFMODULE_MISC2: U6.(INT0)PD2
- new net SENSOR_3V3: J1-1.S, J2-1.S, J3-1.S, R3.2, R4.1, SENSOR_CURRENT.P$2, U1.VDD
- net 3V3: now also C5.2, C6.2, C7.2
- net GND: now also C3.1, C4.1, C5.1, C6.1, C7.1
- net RFMODULE_3V3: now also C3.2, C4.2
- net RFMODULE_MISC2_INT: now also U6.(INT0)PD2
Other:
- note added: "5V (not used)"
- note added: "TODO use electrolytic somewhere nearby"
- note removed: "Note: Arduino power might be higher voltage than 3V3 - should signal 1 to the device by just not driving it low (pullup resistor does the work)."
- note removed: "TODO bigger pads"
